File: PCB/JayKey2.kicad_pcb (KiCad board)
At the start: 4 copper layers, 2 parts, among them U1 ATXMEGA128A1U-AU, U2 RN42

Commit message: 2018.04.30 Update
- Added personal library with LED driver symbols
- Added key switch matrix from JayKey1
- Updated readme to differentiate this keyboard from JayKey1
Parts:
- removed U1: ATXMEGA128A1U-AU, Housings_QFP:TQFP-100_14x14mm_Pitch0.5mm
- removed U2: RN42, keyboard_parts:RN42
